Commit message: Update

File: robots/xpp_hyq/urdf/leg.urdf.xacro (robot description, xacro)
@@ -63,5 +63,7 @@
 					<mesh filename="package://xpp_hyq/meshes/leg/lowerleg.dae" scale="1 1 1"/>
 				</geometry>
-				<material name="white"/>
+				<material name="white">
+					<color rgba="1.0 1.0 1.0 1.0"/>
+				</material>
 			</visual>
 		</link>
