Commit message: Xpp update

File: robots/xpp_hyq/urdf/a1_biped.urdf (robot description, URDF)
Before this commit: robot a1_biped_description, 23 links, 22 joints
Joints:
- joint RL_foot_fixed: axis (none) -> 0 1 0; origin xyz=0 0 -0.2 rpy=0 0 0 -> xyz=0 0 -0.2 rpy=0 0.0 0
- joint RR_foot_fixed: origin xyz=0 0 -0.2 rpy=0 0 0 -> xyz=0 0 -0.2 rpy=0 0.785402 0
